File: hardware/yamabiko_a/yamabiko_a.kicad_pcb (KiCad board)
At the start: 2 copper layers, 68.6 x 53.3 mm, 44 parts, among them J1 MJ-179PH, J101 Power, J102 D8-D13/SDA/SCL, J103 D0-D7, J104 A0-A5, J2 ACTUATOR, J3 FAN, J4 SCS0009, J5 VALVE, Q1 MTB060P06I3, Q2 2N7000, Q3 2N7000, Q4 2SK4017, SW1 EXEC, U1 TB6643KQ, U2 NJM7806FA, U3 74HC125

Commit message: Board name and revision on the silkscreen of both boards
design.py gets REV (1.0) and the name printed on each board; the
schematic title blocks carry the same revision. gen_boards.place_title
puts "Yamabiko No.1 A Rev 1.0" (B likewise) on the front silkscreen at
the free spot nearest the middle of the board, clear of pads, silkscreen,
courtyards and the real outline (sampled against the board polygon, which
matters for the Arduino shape), at the largest size that fits and on two
lines if one does not. add_title.py does the same for an already routed
board, so a new revision does not mean routing again. Both come out at
0.8 mm: A between U1 and R1, B along the bottom edge under R6 / R10.
DRC and ERC are as before.

Co-Authored-By: Claude Opus 5 <noreply@anthropic.com>
Other:
- board text added: "Yamabiko No.1 A Rev 1.0"
Changed lines of the file:
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@@
 		(layer "Edge.Cuts")
+	)
+	(gr_text "Yamabiko No.1 A Rev 1.0"
+		(at 133.475 58.385 0)
+		(layer "F.SilkS")
+		(effects
+			(font
+				(size 0.8 0.8)
+				(thickness 0.12)
+			)
+		)
 	)
 	(segment
