File: hardware/yamabiko_b/yamabiko_b.kicad_pcb (KiCad board)
At the start: 2 copper layers, 40.7 x 53.3 mm, 18 parts, among them J1 MIC1 SAI1 3V3, J14 Carrier J14 (socket, bottom), J15 Carrier J15 (socket, bottom), J2 MIC2 MI2S0 1V8, J3 I2C4 3V3, J4 GPIO 3V3

Commit message: Board name and revision on the silkscreen of both boards
design.py gets REV (1.0) and the name printed on each board; the
schematic title blocks carry the same revision. gen_boards.place_title
puts "Yamabiko No.1 A Rev 1.0" (B likewise) on the front silkscreen at
the free spot nearest the middle of the board, clear of pads, silkscreen,
courtyards and the real outline (sampled against the board polygon, which
matters for the Arduino shape), at the largest size that fits and on two
lines if one does not. add_title.py does the same for an already routed
board, so a new revision does not mean routing again. Both come out at
0.8 mm: A between U1 and R1, B along the bottom edge under R6 / R10.
DRC and ERC are as before.

Co-Authored-By: Claude Opus 5 <noreply@anthropic.com>
Other:
- board text added: "Yamabiko No.1 B Rev 1.0"
Changed lines of the file:
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@@
 		(layer "Edge.Cuts")
+	)
+	(gr_text "Yamabiko No.1 B Rev 1.0"
+		(at 152.57 107.16 0)
+		(layer "F.SilkS")
+		(effects
+			(font
+				(size 0.8 0.8)
+				(thickness 0.12)
+			)
+		)
 	)
 	(segment
